File: pcb_data/Assemble_L/Assemble_L.kicad_sch (KiCad schematic)
At the start: 63 parts, among them SW1 SW_Push, SW10 SW_Push, SW11 SW_Push, SW12 SW_Push, SW13 SW_Push, SW14 SW_Push, SW15 SW_Push, SW16 SW_Push, SW17 SW_Push, SW18 SW_Push, SW19 SW_Push, SW2 SW_Push, SW20 SW_Push, SW21 SW_Push, SW22 SW_Push, SW23 SW_Push, SW24 SW_Push, SW25 SW_Push, SW26 SW_Push, SW27 SW_Push, SW28 SW_Push, SW29 SW_Push, SW3 SW_Push, SW30 SW_Push, SW31 SW_Push, SW4 SW_Push, SW5 SW_Push, SW6 SW_Push, SW7 SW_Push, SW8 SW_Push, SW9 SW_Push, U1 XIAO-HALF-HOLE-23P

Commit message: temp kicad file
Parts:
- removed U1: XIAO-HALF-HOLE-23P, Module:MOUDLE23P-XIAO-HALF-HOLE, symbol MOUDLE-SEEEDUINO-XIAO-ESP32S3-Plus:Module/XIAO-HALF-HOLE-23P
- added LED1, LED2, LED3, LED4: LED_SK6812MINI-E, symbol Salicylic_kbd:LED_SK6812MINI-E
- added U1: ~, symbol Seeed_Studio_XIAO_Series:XIAO-nRF52840_Plus_SMD
Connections:
- net GND: now also LED1.2 (VSS), LED2.2 (VSS), LED3.2 (VSS), LED4.2 (VSS), U1.13 (GND), U1.27 (GND), U1.33 (GND)
- net VCC: now also LED1.4 (VDD), LED2.4 (VDD), LED3.4 (VDD), LED4.4 (VDD), U1.32 (VBAT)
- net at SW16.1: now also SW10.1, SW22.1, SW28.1, SW3.1
- net at D5.1 (K): now also D1.1 (K), D2.1 (K), D3.1 (K), D4.1 (K), D6.1 (K), D7.1 (K)
- net at D18.1 (K): now also D14.1 (K), D15.1 (K), D16.1 (K), D17.1 (K), D19.1 (K)
- net at D25.1 (K): now also D20.1 (K), D21.1 (K), D22.1 (K), D23.1 (K), D24.1 (K)
- net at D30.1 (K): now also D26.1 (K), D27.1 (K), D28.1 (K), D29.1 (K), D31.1 (K)
- net at SW8.1: now also SW1.1, SW14.1, SW20.1, SW26.1
- net at D13.1 (K): now also D10.1 (K), D11.1 (K), D12.1 (K), D8.1 (K), D9.1 (K)
- net at SW2.1: now also SW15.1, SW21.1, SW27.1, SW9.1
- net at SW4.1: now also SW11.1, SW17.1, SW23.1, SW29.1
- net at SW31.1: now also SW13.1, SW19.1, SW25.1, SW6.1
- net at SW18.1: now also SW12.1, SW24.1, SW30.1, SW5.1
- new net: LED3.1 (DOUT), LED4.3 (DIN)
- new net: LED2.1 (DOUT), LED3.3 (DIN)
- new net: LED1.1 (DOUT), LED2.3 (DIN)
Other:
- moved on the sheet: D1, D10, D11, D12, D13, D14, D15, D16, D17, D18, D19, D2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
