File: pcb_data/Assemble_L/Assemble_L.kicad_sch (KiCad schematic)
At the start: 75 parts, among them U1 XIAO-nRF52840-DIP

Commit message: temp kicad file
Parts:
- D0-1, D0-2, D0-3, D0-4, D1-0, D1-2, D1-3, D1-4, D2-0, D2-1, D2-3, D2-4, D3-0, D3-1, D3-2, D3-4, D4-0, D4-1, D4-2, D4-3, D5-0, D5-1, D5-2, D5-3, D5-4, D6-0, D6-1, D6-2, D6-3, D6-4, D6-5, DI0, DI1, DI2, DI3, DI4, DI5, DS0, DS1, DS2, DS3, DS4, DS5: value 1N4148 -> 1N4148W; footprint Diode_THT:D_DO-35_SOD27_P7.62mm_Horizontal -> kbd_Parts:Diode_TH_SMD
- U1: footprint Module:MOUDLE14P-XIAO-DIP-SMD -> Seeed Studio XIAO Series Library:XIAO-nRF52840-DIP
Connections:
- no-connect marks 0 -> 5

Commit message: update symbol
Parts:
- U1: value XIAO-nRF52840-DIP -> XIAO-nRF52840; footprint Seeed Studio XIAO Series Library:XIAO-nRF52840-DIP -> custom-library:XIAO-nRF52840; symbol Seeed_Studio_XIAO_Series:XIAO-nRF52840-DIP -> Seeed_Studio_XIAO_Series:XIAO-nRF52840-SMD
Connections:
- net GND: now also U1.16 (GND), U1.22 (GND)
- new net VCC: U1.15 (BAT)
- no-connect marks 5 -> 10
Other:
- moved on the sheet: D0-1, D0-2, D0-3, D0-4, D1-0, D1-2, D1-3, D1-4, D2-0, D2-1, D2-3, D2-4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
