File: pcb_data/Assemble_L/round-robin-8-42.kicad_sch (KiCad schematic)
At the start: 99 parts, among them U2 XIAO-nRF52840-SMD

Commit message: temp kicad file
Parts:
- removed D32, D33, D34, D35, D36, D37, D38, D39, D40, D41, D42, D43, D44, D45, D46, D47, D48, D49, D50, D51: 1N4148, Diode_THT:D_DO-35_SOD27_P7.62mm_Horizontal, symbol Diode:1N4148
- removed U2: XIAO-nRF52840-SMD, symbol 17q5doE69gfxD-JFbVQb6s-cbEHCa-Cq-:XIAO-nRF52840-SMD
- added D1, D10, D12, D13, D14, D15, D16, D2, D20, D21, D23, D24, D25, D26, D3, D30, D31, D4, D5, D6: 1N4148, Diode_THT:D_DO-35_SOD27_P7.62mm_Horizontal, symbol Diode:1N4148
Connections:
- net at D32.1 (K), D42.1 (K), D52.1 (K)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: now also D12.1 (K), D2.1 (K)
- net at D41.1 (K), D51.1 (K), D61.1 (K)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: now also D1.1 (K), D21.1 (K), D31.1 (K)
- net at D40.1 (K), D50.1 (K), D60.1 (K)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: now also D10.1 (K), D20.1 (K), D30.1 (K)
- net at RC1-0.2: now also D10.2 (A)
- net at D35.1 (K), D45.1 (K), D65.1 (K)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: now also D15.1 (K), D25.1 (K), D5.1 (K)
- net at D36.1 (K), D46.1 (K), D56.1 (K)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: now also D16.1 (K), D26.1 (K), D6.1 (K)
- net at RC3-0.2: now also D30.2 (A)
- net at RC3-1.2: now also D31.2 (A)
- net at RC2-3.2: now also D23.2 (A)
- net at D43.1 (K), D53.1 (K), D63.1 (K)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: now also D13.1 (K), D23.1 (K), D3.1 (K)
- net at RC1-2.2: now also D12.2 (A)
- net at RC1-3.2: now also D13.2 (A)
- net at RC1-4.2: now also D14.2 (A)
- net at D34.1 (K), D54.1 (K), D64.1 (K)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: now also D14.1 (K), D24.1 (K), D4.1 (K)
- net at RC2-6.2: now also D26.2 (A)
- net at RC0-1.2: now also D1.2 (A)
- net at RC0-2.2: now also D2.2 (A)
- net at RC1-6.2: now also D16.2 (A)
- net at RC2-4.2: now also D24.2 (A)
- net at RC0-5.2: now also D5.2 (A)
- net at RC2-0.2: now also D20.2 (A)
- net at RC0-4.2: now also D4.2 (A)
- net at RC1-5.2: now also D15.2 (A)
- net at RC2-1.2: now also D21.2 (A)
- net at RC0-3.2: now also D3.2 (A)
- net at RC2-5.2: now also D25.2 (A)
- net at RC0-6.2: now also D6.2 (A)
Other:
- moved on the sheet: D32, D34, D35, D36, D40, D41, D42, D43, D45, D46, D50, D51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
