File: pcb_data/Assemble/Assemble.kicad_sch (KiCad schematic)
At the start: 198 parts, among them U1 XIAO-nRF52840-SMD, U2 XIAO-nRF52840-SMD

Commit message: temp kicad file
Parts:
- U1, U2: footprint (none) -> Seeed Studio XIAO Series Library:XIAO-nRF52840-SMD
Changed lines of the file:
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@@
 			)
 		)
-		(property "Footprint" ""
+		(property "Footprint" "Seeed Studio XIAO Series Library:XIAO-nRF52840-SMD"
 			(at 111.76 40.64 0)
 			(effects
@@
 			)
 		)
-		(property "Footprint" ""
+		(property "Footprint" "Seeed Studio XIAO Series Library:XIAO-nRF52840-SMD"
 			(at 247.65 40.64 0)
 			(effects

Commit message: temp kicad file
Parts:
- RC0-1: footprint (none) -> Kailh_PG1353_Hotswap:Kailh-PG1353-Hotswap-1.5U
- RC0-10, RC0-11, RC0-13, RC0-4, RC0-5, RC0-6, RC0-8, RC0-9, RC1-0, RC1-10, RC1-11, RC1-12, RC1-13, RC1-2, RC1-3, RC1-4, RC1-5, RC1-6, RC1-7, RC1-9, RC2-0, RC2-1, RC2-10, RC2-11, RC2-12, RC2-13, RC2-3, RC2-4, RC2-5, RC2-6, RC2-7, RC2-8, RC3-0, RC3-1, RC3-11, RC3-12, RC3-13, RC3-2, RC3-4, RC3-5, RC3-6, RC3-7, RC3-8, RC3-9, RC4-0, RC4-1, RC4-10, RC4-12, RC4-13, RC4-2, RC4-3, RC4-5, RC4-6, RC4-7, RC4-8, RC4-9, RC5-0, RC5-1, RC5-10, RC5-11, RC5-13, RC5-2, RC5-3, RC5-4, RC5-6, RC5-7, RC5-8, RC5-9, RC6-0, RC6-1, RC6-10, RC6-11, RC6-12, RC6-2, RC6-3, RC6-4, RC6-7, RC6-8: footprint (none) -> Kailh_PG1353_Hotswap:Kailh-PG1353-Hotswap-1U
- RC0-12, RC6-5: footprint (none) -> Kailh_PG1353_Hotswap:Kailh-PG1353-Hotswap-1.25U
- RC0-2: footprint (none) -> Kailh_PG1353_Hotswap:Kailh-PG1353-Hotswap-1.75U
- RC0-3, RC6-9: footprint (none) -> Kailh_PG1353_Hotswap:Kailh-PG1353-Hotswap-2U

Commit message: temp kicad file
Parts:
- removed D15, D16, D18, D25, D26, D33, D35, D36, D45, D46, D48, D5, D56, D6, DI6, DS6: 1N4148, Diode_THT:D_DO-35_SOD27_P7.62mm_Horizontal, symbol Diode:1N4148
- removed RC0-13, RC0-5, RC0-6, RC1-13, RC1-5, RC1-6, RC2-13, RC2-5, RC2-6, RC3-5, RC3-6, RC4-5, RC4-6, RC5-6: SW_Push, Kailh_PG1353_Hotswap:Kailh-PG1353-Hotswap-1U, symbol Switch:SW_Push

Commit message: temp kicad file
Parts:
- RC6-9: footprint Kailh_PG1353_Hotswap:Kailh-PG1353-Hotswap-2U -> Kailh_PG1353_Hotswap:Kailh-PG1353-Hotswap-1.5U
- U1, U2: footprint Seeed Studio XIAO Series Library:XIAO-nRF52840-SMD -> Seeed Studio XIAO Series Library:XIAO-nRF52840-DIP
Changed lines of the file:
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@@
 	)
 	(symbol
+		(lib_name "XIAO-nRF52840-SMD_1")
 		(lib_id "Seeed_Studio_XIAO_Series:XIAO-nRF52840-SMD")
 		(at 120.65 45.72 0)
@@
 			)
 		)
-		(property "Footprint" "Seeed Studio XIAO Series Library:XIAO-nRF52840-SMD"
+		(property "Footprint" "Seeed Studio XIAO Series Library:XIAO-nRF52840-DIP"
 			(at 111.76 40.64 0)
 			(effects
@@
 		(pin "10"
 		)
-		(pin "34"
-		)
-		(pin "32"
+		(pin "15"
+		)
+		(pin "19"
 		)
 		(pin "5"
@@
 		(pin "3"
 		)
-		(pin "25"
-		)
-		(pin "26"
+		(pin "16"
+		)
+		(pin "20"
 		)
 		(pin "14"
@@
 		(pin "13"
 		)
-		(pin "35"
-		)
-		(pin "27"
+		(pin "21"
+		)
+		(pin "17"
 		)
 		(pin "12"
@@
 		(pin "8"
 		)
-		(pin "33"
+		(pin "22"
 		)
 		(pin "6"
 		)
-		(pin "24"
+		(pin "18"
 		)
 		(pin "1"
@@
 			)
 		)
-		(property "Footprint" "Seeed Studio XIAO Series Library:XIAO-nRF52840-SMD"
+		(property "Footprint" "Seeed Studio XIAO Series Library:XIAO-nRF52840-DIP"
 			(at 247.65 40.64 0)
 			(effects
@@
 		(pin "10"
 		)
-		(pin "34"
-		)
-		(pin "32"
+		(pin "19"
+		)
+		(pin "16"
 		)
 		(pin "5"
@@
 		(pin "3"
 		)
-		(pin "25"
-		)
-		(pin "26"
+		(pin "20"
+		)
+		(pin "21"
 		)
 		(pin "14"
@@
 		(pin "13"
 		)
-		(pin "35"
-		)
-		(pin "27"
+		(pin "17"
+		)
+		(pin "22"
 		)
 		(pin "12"
@@
 		(pin "8"
 		)
-		(pin "33"
+		(pin "18"
 		)
 		(pin "6"
 		)
-		(pin "24"
+		(pin "15"
 		)
 		(pin "1"
@@
 			)
 		)
-		(property "Footprint" "Kailh_PG1353_Hotswap:Kailh-PG1353-Hotswap-2U"
+		(property "Footprint" "Kailh_PG1353_Hotswap:Kailh-PG1353-Hotswap-1.5U"
 			(at 355.6 154.94 0)
 			(effects

Commit message: temp kicad file
Parts:
- RC6-9: footprint Kailh_PG1353_Hotswap:Kailh-PG1353-Hotswap-1.5U -> 0temp-library:Kailh-PG1353-Hotswap-ISOEnter
Changed lines of the file:
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@@
 			)
 		)
-		(property "Footprint" "Kailh_PG1353_Hotswap:Kailh-PG1353-Hotswap-1.5U"
+		(property "Footprint" "0temp-library:Kailh-PG1353-Hotswap-ISOEnter"
 			(at 355.6 154.94 0)
 			(effects

Commit message: temp
Parts:
- renumbered D1 to D0-1, D9 to D0-10, D11 to D0-11, D17 to D0-12, D2 to D0-2, D3 to D0-3, D4 to D0-4, D7 to D0-8, D8 to D0-9, D10 to D1-0, D27 to D1-10, D28 to D1-11, D29 to D1-12, D12 to D1-2, D13 to D1-3, D14 to D1-4, D19 to D1-7, D22 to D1-9, D20 to D2-0, D21 to D2-1, D39 to D2-10, D44 to D2-11, D47 to D2-12, D23 to D2-3, D24 to D2-4, D37 to D2-7, D38 to D2-8, D30 to D3-0, D31 to D3-1, D58 to D3-11, D59 to D3-12, D66 to D3-13, D32 to D3-2, D34 to D3-4, D49 to D3-7, D55 to D3-8, D57 to D3-9, D40 to D4-0, D41 to D4-1, D70 to D4-10, D71 to D4-12, D72 to D4-13, D42 to D4-2, D43 to D4-3, D67 to D4-7, D68 to D4-8, D69 to D4-9, D50 to D5-0, D51 to D5-1, D76 to D5-10, D77 to D5-11, D78 to D5-13, D52 to D5-2, D53 to D5-3, D54 to D5-4, D73 to D5-7, D74 to D5-8, D75 to D5-9, D60 to D6-0, D61 to D6-1, D82 to D6-10, D83 to D6-11, D84 to D6-12, D62 to D6-2, D63 to D6-3, D64 to D6-4, D65 to D6-5, D79 to D6-7, D80 to D6-8, D81 to D6-9
Connections:
- net GND: now reaches U1.13 (GND)
- net GND: now also U2.13 (GND)
- no-connect marks 0 -> 10
