File: pcb_data/Assemble_R/Assemble_R.kicad_sch (KiCad schematic)
At the start: 93 parts, among them U1 XIAO-nRF52840-DIP

Commit message: update symbol
Parts:
- U1: value XIAO-nRF52840-DIP -> XIAO-nRF52840; footprint Seeed Studio XIAO Series Library:XIAO-nRF52840-DIP -> custom-library:XIAO-nRF52840; symbol Seeed_Studio_XIAO_Series:XIAO-nRF52840-DIP -> Seeed_Studio_XIAO_Series:XIAO-nRF52840-SMD
Connections:
- net GND: now also U1.16 (GND), U1.22 (GND)
- new net VCC: U1.15 (BAT)
- no-connect marks 5 -> 10
Other:
- moved on the sheet: U1

Commit message: Update right sch
Parts:
- RC0-12: footprint Kailh_PG1353_Hotswap:Kailh-PG1353-Hotswap-1.25U -> Kailh_PG1353_Hotswap:Kailh-PG1353-Hotswap-1U
- RC0-13: renamed from RC6-7; footprint Kailh_PG1353_Hotswap:Kailh-PG1353-Hotswap-1U -> Kailh_PG1353_Hotswap:Kailh-PG1353-Hotswap-1.25U
- RC6-10: footprint Kailh_PG1353_Hotswap:Kailh-PG1353-Hotswap-1U -> custom-library:Kailh-PG1353-Hotswap-ISOEnter
- RC6-9: footprint custom-library:Kailh-PG1353-Hotswap-ISOEnter -> Kailh_PG1353_Hotswap:Kailh-PG1353-Hotswap-1U
- renumbered D6-7 to D0-13, D4-13 to D2-13, RC4-13 to RC2-13
Connections:
- net IO 11: no longer RC2-13.1
- net IO 13: no longer RC0-13.1
- net IO 7: now also RC0-13.1
- net IO 9: now also RC2-13.1
- net at D1-7.1 (K), D2-7.1 (K), D3-7.1 (K)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: no longer D0-13.1 (K)
- net at D2-13.1 (K), D3-13.1 (K), D5-13.1 (K)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: now also D0-13.1 (K)
Other:
- moved on the sheet: D0-13, D2-13, RC0-13, RC2-13
