File: pcb_data/Assemble_R/Assemble_R.kicad_pcb (KiCad board)
At the start: 2 copper layers, 93 parts, among them U1 XIAO-nRF52840-DIP

Commit message: temp kicad file
Other:
- board outline added: 204.8 x 109.5 mm
Changed lines of the file:
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@@
 		)
+	)
+	(gr_line
+		(start 221.45625 150.01875)
+		(end 221.45625 76.2)
+		(stroke
+			(width 0.05)
+			(type default)
+		)
+		(layer "Edge.Cuts")
+	)
+	(gr_line
+		(start 42.8625 40.48125)
+		(end 42.8625 150.01875)
+		(stroke
+			(width 0.05)
+			(type default)
+		)
+		(layer "Edge.Cuts")
+	)
+	(gr_line
+		(start 221.45625 76.2)
+		(end 247.65 76.2)
+		(stroke
+			(width 0.05)
+			(type default)
+		)
+		(layer "Edge.Cuts")
+	)
+	(gr_line
+		(start 247.65 40.48125)
+		(end 42.8625 40.48125)
+		(stroke
+			(width 0.05)
+			(type default)
+		)
+		(layer "Edge.Cuts")
+	)
+	(gr_line
+		(start 247.65 76.2)
+		(end 247.65 40.48125)
+		(stroke
+			(width 0.05)
+			(type default)
+		)
+		(layer "Edge.Cuts")
+	)
+	(gr_line
+		(start 42.8625 150.01875)
+		(end 221.45625 150.01875)
+		(stroke
+			(width 0.05)
+			(type default)
+		)
+		(layer "Edge.Cuts")
 	)
 	(embedded_fonts no)

Commit message: temp kicad file
Parts:
- moved DI8 32.4 mm to (164.3, 81.0)
- moved DI7 19.2 mm to (173.8, 61.9)
- moved DI9 13.5 mm to (190.5, 81.0)
- moved D2-11 4.76 mm to (121.4, 119.1)
- moved D5-9 4.76 mm to (169.1, 81.0)
Routing:
- net IO 10: track 0.00 -> 267.9 mm, vias 0 -> 14
- net IO 7: track 0.00 -> 253.8 mm, vias 0 -> 7
- net IO 9: track 0.00 -> 248.5 mm, vias 0 -> 7
- net IO 11: track 0.00 -> 223.6 mm, vias 0 -> 10
- net IO 8: track 0.00 -> 219.8 mm, vias 0 -> 7
- net IO 12: track 0.00 -> 206.1 mm, vias 0 -> 9
- net Net-(D0-12-K): track 0.00 -> 193.2 mm, vias 0 -> 1
- net IO 13: track 0.00 -> 192.8 mm, vias 0 -> 5
- net Net-(D0-9-K): track 0.00 -> 181.0 mm
- net Net-(D0-10-K): track 0.00 -> 171.2 mm
- net Net-(D0-11-K): track 0.00 -> 168.9 mm, vias 0 -> 2
- net INTR_R: track 0.00 -> 163.3 mm, vias 0 -> 4
- net Net-(D0-8-K): track 0.00 -> 153.5 mm
- net Net-(D1-7-K): track 0.00 -> 137.2 mm
- net Net-(D3-13-K): track 0.00 -> 114.9 mm
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
Commit message: update symbol
Parts:
- U1: value XIAO-nRF52840-DIP -> XIAO-nRF52840; footprint Seeed Studio XIAO Series Library:XIAO-nRF52840-DIP -> custom-library:XIAO-nRF52840
Changed lines of the file:
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@@
 	(net 53 "IO 12")
 	(net 54 "IO 13")
-	(net 55 "unconnected-(U1-P1.15_MOSI_D10-Pad11)")
-	(net 56 "unconnected-(U1-3V3-Pad12)")
-	(net 57 "unconnected-(U1-P1.14_MISO_D9-Pad10)")
-	(net 58 "unconnected-(U1-VBUS-Pad14)")
-	(net 59 "unconnected-(U1-P1.13_SCK_D8-Pad9)")
-	(net 60 "unconnected-(U1-3V3-Pad12)_1")
-	(net 61 "unconnected-(U1-P1.14_MISO_D9-Pad10)_1")
-	(net 62 "GND")
-	(net 63 "unconnected-(U1-VBUS-Pad14)_1")
-	(net 64 "unconnected-(U1-P1.13_SCK_D8-Pad9)_1")
-	(net 65 "unconnected-(U1-P1.15_MOSI_D10-Pad11)_1")
+	(net 55 "unconnected-(U1-3V3-Pad12)")
+	(net 56 "unconnected-(U1-3V3-Pad12)_1")
+	(net 57 "GND")
+	(net 58 "unconnected-(U1-P1.14_D9_MISO-Pad10)")
+	(net 59 "unconnected-(U1-P1.14_D9_MISO-Pad10)_1")
+	(net 60 "unconnected-(U1-P1.13_D8_SCK-Pad9)")
+	(net 61 "unconnected-(U1-P1.13_D8_SCK-Pad9)_1")
+	(net 62 "unconnected-(U1-PA31_SWDIO-Pad19)")
+	(net 63 "unconnected-(U1-PA30_SWCLK-Pad20)")
+	(net 64 "VCC")
+	(net 65 "unconnected-(U1-RESET-Pad21)")
+	(net 66 "unconnected-(U1-5V-Pad14)")
+	(net 67 "unconnected-(U1-5V-Pad14)_1")
+	(net 68 "unconnected-(U1-P1.15_D10_MOSI-Pad11)")
+	(net 69 "unconnected-(U1-P1.15_D10_MOSI-Pad11)_1")
+	(net 70 "unconnected-(U1-NFC2-Pad18)")
+	(net 71 "unconnected-(U1-NFC1-Pad17)")
 	(footprint "kbd_Parts:Diode_TH_SMD"
 		(layer "F.Cu")
@@
 		)
 	)
-	(footprint "Seeed Studio XIAO Series Library:XIAO-nRF52840-DIP"
+	(footprint "custom-library:XIAO-nRF52840"
 		(layer "F.Cu")
 		(at 230.505 59.84875)
@@
 			)
 		)
-		(property "Value" "XIAO-nRF52840-DIP"
-			(at 0 0 0)
+		(property "Value" "XIAO-nRF52840"
+			(at 0.055 6.5 0)
 			(unlocked yes)
 			(layer "F.Fab")
@@
 			(end -6.985 -10.541)
 			(stroke
-				(width 0.1)
-				(type solid)
-			)
-			(layer "F.SilkS")
-		)
-		(fp_line
-			(start 6.985 -10.541)
-			(end -6.985 -10.541)
-			(stroke
 				(width 0.127)
 				(type solid)
@@
 			(roundrect_rratio 0.1)
 			(net 47 "INTR_R")
-			(pinfunction "P0.02_AIN0_LOW_A0_D0")
+			(pinfunction "P0.02_A0_D0")
 			(pintype "passive")
 			(thermal_bridge_angle 45)
@@
 			(remove_unused_layers no)
 			(net 47 "INTR_R")
-			(pinfunction "P0.02_AIN0_LOW_A0_D0")
+			(pinfunction "P0.02_A0_D0")
 			(pintype "passive")
 		)
@@
 			(roundrect_rratio 0.1)
 			(net 48 "IO 7")
-			(pinfunction "P0.03_AIN1_LOW_A1_D1")
+			(pinfunction "P0.03_A1_D1")
 			(pintype "passive")
 			(thermal_bridge_angle 45)
@@
 			(remove_unused_layers no)
 			(net 48 "IO 7")
-			(pinfunction "P0.03_AIN1_LOW_A1_D1")
+			(pinfunction "P0.03_A1_D1")
 			(pintype "passive")
 		)
@@
 			(roundrect_rratio 0.1)
 			(net 49 "IO 8")
-			(pinfunction "P0.28_AIN4_LOW_A2_D2")
+			(pinfunction "P0.28_A2_D2")
 			(pintype "passive")
 			(thermal_bridge_angle 45)
@@
 			(remove_unused_layers no)
 			(net 49 "IO 8")
-			(pinfunction "P0.28_AIN4_LOW_A2_D2")
+			(pinfunction "P0.28_A2_D2")
 			(pintype "passive")
 		)
@@
 			(roundrect_rratio 0.1)
 			(net 50 "IO 9")
-			(pinfunction "P0.29_AIN5_LOW_A3_D3")
+			(pinfunction "P0.29_A3_D3")
 			(pintype "passive")
 			(thermal_bridge_angle 45)
@@
 			(remove_unused_layers no)
 			(net 50 "IO 9")
-			(pinfunction "P0.29_AIN5_LOW_A3_D3")
+			(pinfunction "P0.29_A3_D3")
 			(pintype "passive")
 		)
@@
 			(roundrect_rratio 0.1)
 			(net 51 "IO 10")
-			(pinfunction "P0.04_AIN2_A4_D4")
+			(pinfunction "P0.04_A4_D4_SDA")
 			(pintype "passive")
 			(thermal_bridge_angle 45)
@@
 			(remove_unused_layers no)
 			(net 51 "IO 10")
-			(pinfunction "P0.04_AIN2_A4_D4")
+			(pinfunction "P0.04_A4_D4_SDA")
 			(pintype "passive")
 		)
@@
 			(roundrect_rratio 0.1)
 			(net 52 "IO 11")
-			(pinfunction "P0.05_AIN3_A5_D5")
+			(pinfunction "P0.05_A5_D5_SCL")
 			(pintype "passive")
 			(thermal_bridge_angle 45)
@@
 			(remove_unused_layers no)
 			(net 52 "IO 11")
-			(pinfunction "P0.05_AIN3_A5_D5")
+			(pinfunction "P0.05_A5_D5_SCL")
 			(pintype "passive")
 		)
@@
 			(roundrect_rratio 0.1)
 			(net 53 "IO 12")
-			(pinfunction "P1.11_TX_D6")
+			(pinfunction "P1.11_D6_TX")
 			(pintype "passive")
 			(thermal_bridge_angle 45)
@@
 			(remove_unused_layers no)
 			(net 53 "IO 12")
-			(pinfunction "P1.11_TX_D6")
+			(pinfunction "P1.11_D6_TX")
 			(pintype "passive")
 		)
@@
 			(remove_unused_layers no)
 			(net 54 "IO 13")
-			(pinfunction "P1.12_RX_D7")
+			(pinfunction "P1.12_D7_RX")
 			(pintype "passive")
 		)
@@
 			(roundrect_rratio 0.1)
 			(net 54 "IO 13")
-			(pinfunction "P1.12_RX_D7")
+			(pinfunction "P1.12_D7_RX")
 			(pintype "passive")
 			(thermal_bridge_angle 45)
@@
 			(layers "*.Cu" "*.Mask")
 			(remove_unused_layers no)
-			(net 59 "unconnected-(U1-P1.13_SCK_D8-Pad9)")
-			(pinfunction "P1.13_SCK_D8")
+			(net 61 "unconnected-(U1-P1.13_D8_SCK-Pad9)_1")
+			(pinfunction "P1.13_D8_SCK")
 			(pintype "passive+no_connect")
 		)
@@
 			(layers "F.Cu" "F.Mask")
 			(roundrect_rratio 0.1)
-			(net 64 "unconnected-(U1-P1.13_SCK_D8-Pad9)_1")
-			(pinfunction "P1.13_SCK_D8")
+			(net 60 "unconnected-(U1-P1.13_D8_SCK-Pad9)")
+			(pinfunction "P1.13_D8_SCK")
 			(pintype "passive+no_connect")
 			(thermal_bridge_angle 45)
@@
 			(layers "*.Cu" "*.Mask")
 			(remove_unused_layers no)
-			(net 57 "unconnected-(U1-P1.14_MISO_D9-Pad10)")
-			(pinfunction "P1.14_MISO_D9")
+			(net 58 "unconnected-(U1-P1.14_D9_MISO-Pad10)")
+			(pinfunction "P1.14_D9_MISO")
 			(pintype "passive+no_connect")
 		)
@@
 			(layers "F.Cu" "F.Mask")
 			(roundrect_rratio 0.1)
-			(net 61 "unconnected-(U1-P1.14_MISO_D9-Pad10)_1")
-			(pinfunction "P1.14_MISO_D9")
+			(net 59 "unconnected-(U1-P1.14_D9_MISO-Pad10)_1")
+			(pinfunction "P1.14_D9_MISO")
 			(pintype "passive+no_connect")
 			(thermal_bridge_angle 45)
@@
 			(layers "*.Cu" "*.Mask")
 			(remove_unused_layers no)
-			(net 65 "unconnected-(U1-P1.15_MOSI_D10-Pad11)_1")
-			(pinfunction "P1.15_MOSI_D10")
+			(net 68 "unconnected-(U1-P1.15_D10_MOSI-Pad11)")
+			(pinfunction "P1.15_D10_MOSI")
 			(pintype "passive+no_connect")
 		)
@@
 			(layers "F.Cu" "F.Mask")
 			(roundrect_rratio 0.1)
-			(net 55 "unconnected-(U1-P1.15_MOSI_D10-Pad11)")
-			(pinfunction "P1.15_MOSI_D10")
+			(net 69 "unconnected-(U1-P1.15_D10_MOSI-Pad11)_1")
+			(pinfunction "P1.15_D10_MOSI")
 			(pintype "passive+no_connect")
 			(thermal_bridge_angle 45)
@@
 			(layers "*.Cu" "*.Mask")
 			(remove_unused_layers no)
-			(net 60 "unconnected-(U1-3V3-Pad12)_1")
+			(net 55 "unconnected-(U1-3V3-Pad12)")
 			(pinfunction "3V3")
 			(pintype "passive+no_connect")
@@
 			(layers "F.Cu" "F.Mask")
 			(roundrect_rratio 0.1)
-			(net 56 "unconnected-(U1-3V3-Pad12)")
+			(net 56 "unconnected-(U1-3V3-Pad12)_1")
 			(pinfunction "3V3")
 			(pintype "passive+no_connect")
@@
 			(layers "*.Cu" "*.Mask")
 			(remove_unused_layers no)
-			(net 62 "GND")
+			(net 57 "GND")
 			(pinfunction "GND")
 			(pintype "passive")
@@
 			(layers "F.Cu" "F.Mask")
 			(roundrect_rratio 0.1)
-			(net 62 "GND")
+			(net 57 "GND")
 			(pinfunction "GND")
 			(pintype "passive")
@@
 			(layers "*.Cu" "*.Mask")
 			(remove_unused_layers no)
-			(net 63 "unconnected-(U1-VBUS-Pad14)_1")
-			(pinfunction "VBUS")
+			(net 66 "unconnected-(U1-5V-Pad14)")
+			(pinfunction "5V")
 			(pintype "passive+no_connect")
 		)
@@
 			(layers "F.Cu" "F.Mask")
 			(roundrect_rratio 0.1)
-			(net 58 "unconnected-(U1-VBUS-Pad14)")
-			(pinfunction "VBUS")
+			(net 67 "unconnected-(U1-5V-Pad14)_1")
+			(pinfunction "5V")
+			(pintype "passive+no_connect")
+			(thermal_bridge_angle 45)
+		)
+		(pad "15" smd roundrect
+			(at -4.5 -0.3135 180)
+			(size 2.5 1.1)
+			(layers "F.Cu" "F.Mask" "F.Paste")
+			(roundrect_rratio 0.25)
+			(net 64 "VCC")
+			(pinfunction "BAT")
+			(pintype "passive")
+			(solder_mask_margin 0.0508)
+			(thermal_bridge_angle 45)
+		)
+		(pad "16" smd roundrect
+			(at -4.5 -2.2185 180)
+			(size 2.5 1.1)
+			(layers "F.Cu" "F.Mask" "F.Paste")
+			(roundrect_rratio 0.25)
+			(net 57 "GND")
+			(pinfunction "GND")
+			(pintype "passive")
+			(solder_mask_margin 0.0508)
+			(thermal_bridge_angle 45)
+		)
+		(pad "17" smd roundrect
+			(at 3.755 9.2369 270)
+			(size 2.5 1.1)
+			(layers "F.Cu" "F.Mask" "F.Paste")
+			(roundrect_rratio 0.25)
+			(net 71 "unconnected-(U1-NFC1-Pad17)")
+			(pinfunction "NFC1")
 			(pintype "passive+no_connect")
+			(solder_mask_margin 0.0508)
 			(thermal_bridge_angle 45)
 		)
+		(pad "18" smd roundrect
+			(at 5.66 9.2369 270)
+			(size 2.5 1.1)
+			(layers "F.Cu" "F.Mask" "F.Paste")
+			(roundrect_rratio 0.25)
+			(net 70 "unconnected-(U1-NFC2-Pad18)")
+			(pinfunction "NFC2")
+			(pintype "passive+no_connect")
+			(solder_mask_margin 0.0508)
+			(thermal_bridge_angle 45)
+		)
+		(pad "19" smd circle
+			(at -1.325 -8.5685)
+			(size 1.7 1.7)
+			(layers "F.Cu" "F.Mask" "F.Paste")
+			(net 62 "unconnected-(U1-PA31_SWDIO-Pad19)")
+			(pinfunction "PA31_SWDIO")
+			(pintype "passive+no_connect")
+		)
+		(pad "20" smd circle
+			(at 1.215 -8.5685)
+			(size 1.7 1.7)
+			(layers "F.Cu" "F.Mask" "F.Paste")
+			(net 63 "unconnected-(U1-PA30_SWCLK-Pad20)")
+			(pinfunction "PA30_SWCLK")
+			(pintype "passive+no_connect")
+		)
+		(pad "21" smd circle
+			(at -1.325 -6.0285)
+			(size 1.7 1.7)
+			(layers "F.Cu" "F.Mask" "F.Paste")
+			(net 65 "unconnected-(U1-RESET-Pad21)")
+			(pinfunction "RESET")
+			(pintype "passive+no_connect")
+		)
+		(pad "22" smd circle
+			(at 1.215 -6.0285)
+			(size 1.7 1.7)
+			(layers "F.Cu" "F.Mask" "F.Paste")
+			(net 57 "GND")
+			(pinfunction "GND")
+			(pintype "passive")
+		)
 		(embedded_fonts no)

Commit message: reset right
Routing:
- net IO 10: track 267.9 -> 0.00 mm, vias 14 -> 0
- net IO 7: track 253.8 -> 0.00 mm, vias 7 -> 0
- net IO 9: track 248.5 -> 0.00 mm, vias 7 -> 0
- net IO 11: track 223.6 -> 0.00 mm, vias 10 -> 0
- net IO 8: track 219.8 -> 0.00 mm, vias 7 -> 0
- net IO 12: track 206.1 -> 0.00 mm, vias 9 -> 0
- net Net-(D0-12-K): track 193.2 -> 0.00 mm, vias 1 -> 0
- net IO 13: track 192.8 -> 0.00 mm, vias 5 -> 0
- net Net-(D0-9-K): track 181.0 -> 0.00 mm
- net Net-(D0-10-K): track 171.2 -> 0.00 mm
- net Net-(D0-11-K): track 168.9 -> 0.00 mm, vias 2 -> 0
- net INTR_R: track 163.3 -> 0.00 mm, vias 4 -> 0
- net Net-(D0-8-K): track 153.5 -> 0.00 mm
- net Net-(D1-7-K): track 137.2 -> 0.00 mm
- net Net-(D3-13-K): track 114.9 -> 0.00 mm
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
Commit message: Update right pcb
Parts:
- removed D4-13, D6-7: 1N4148W, kbd_Parts:Diode_TH_SMD
- removed RC4-13, RC6-7: SW_Push, Kailh_PG1353_Hotswap:Kailh-PG1353-Hotswap-1U
- added D0-13: 1N4148W, kbd_Parts:Diode_TH_SMD, F.Cu at (69.1, 133.3)
- added D2-13: 1N4148W, kbd_Parts:Diode_TH_SMD, F.Cu at (109.5, 133.3)
- added RC0-13: SW_Push, Kailh_PG1353_Hotswap:Kailh-PG1353-Hotswap-1.25U, B.Cu at (76.2, 133.3)
- added RC2-13: SW_Push, Kailh_PG1353_Hotswap:Kailh-PG1353-Hotswap-1U, B.Cu at (116.7, 133.3)
- RC0-12: footprint Kailh_PG1353_Hotswap:Kailh-PG1353-Hotswap-1.25U -> Kailh_PG1353_Hotswap:Kailh-PG1353-Hotswap-1U
- RC6-10: footprint Kailh_PG1353_Hotswap:Kailh-PG1353-Hotswap-1U -> custom-library:Kailh-PG1353-Hotswap-ISOEnter; moved to F.Cu
- RC6-9: footprint custom-library:Kailh-PG1353-Hotswap-ISOEnter -> Kailh_PG1353_Hotswap:Kailh-PG1353-Hotswap-1U; moved to B.Cu
- moved DS7 132.4 mm to (196.5, 65.5), turned to 180 degrees
- moved DS9 116.2 mm to (206.0, 71.4), turned to 180 degrees
- moved DS8 116.2 mm to (203.6, 67.9), turned to 180 degrees
- moved DS10 100.6 mm to (207.2, 75.0), turned to 180 degrees
- moved DI8 69.8 mm to (234.0, 85.7), turned to 180 degrees
- moved DS11 66.3 mm to (217.3, 95.2), turned to 180 degrees
- moved DI7 62.1 mm to (234.0, 77.4), turned to 180 degrees
- moved DS12 60.1 mm to (220.3, 100.0), turned to 180 degrees
- moved D2-12 58.0 mm to (152.4, 114.3)
- moved RC2-12 58.0 mm to (159.5, 114.3)
- moved DI9 45.4 mm to (234.0, 94.1), turned to 180 degrees
- moved DI10 38.8 mm to (234.0, 102.4), turned to 180 degrees
- moved DI11 35.8 mm to (234.6, 109.5), turned to 180 degrees
- moved D6-10 34.8 mm to (207.2, 85.1)
- moved RC6-10 34.7 mm to (214.3, 85.7), turned to 0 degrees
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Other:
- board size 204.8 x 109.5 mm -> 238.1 x 131 mm
